File: NoodleDriver/power.kicad_sch (KiCad schematic)
At the start: 11 parts, among them J4 Conn_01x02_Socket, U5 TP4057, U7 DS8242-33S3

Commit message: Final tuning of prototype board, which we've ordered a handful of prototypes to be fabbed.  Part of #8
Parts:
- added Q1: JSM2302, Package_TO_SOT_SMD:SOT-23, symbol Transistor_FET:DMN2041L
- added R10: 10K, Resistor_SMD:R_0402_1005Metric, symbol Device:R_Small
- added R14: 100K, Resistor_SMD:R_0402_1005Metric, symbol Device:R_Small
- added SW1: On/Off, Button_Switch_THT:SW_Slide_SPDT_Angled_CK_OS102011MA1Q, symbol Switch:SW_SPDT
Connections:
- net +3V3: now also R10.1
- net GND: now also Q1.3 (D); no longer C3.2, C4.2, J4.2 (Pin_2), R11.2, U5.2 (GND)
- new net: R10.2, SW1.2 (B)
- new net: Q1.1 (G), R14.1, SW1.3 (C)
- new net -BATT: C3.2, C4.2, J4.2 (Pin_2), Q1.2 (S), R11.2, R14.2, U5.2 (GND)
- no-connect marks 0 -> 1
